Commit message: 0522 RL 추가

File: isaaclab_real/complete_asm/complete_asm.urdf (robot description, URDF)
Before this commit: robot complete_asm, 8 links, 17 joints
Links:
- removed link LOWER_ARM_LINK미러
- removed link TOP_ARM_LINK미러
- added link LOWER_ARM_LINK_MIR, mass 0.07644747488590391; collision mesh filename=meshes/LOWER_ARM_LINK_MIR.stl scale=0.001 0.001 0.001; visual mesh filename=meshes/LOWER_ARM_LINK_MIR.stl scale=0.001 0.001 0.001
- added link TOP_ARM_LINK_MIR, mass 0.1912083481787344; collision mesh filename=meshes/TOP_ARM_LINK_MIR.stl scale=0.001 0.001 0.001; visual mesh filename=meshes/TOP_ARM_LINK_MIR.stl scale=0.001 0.001 0.001
Joints:
- removed joint BODY_LINK_회전-18
- removed joint LOWER_ARM_LINK_회전-8
- removed joint LOWER_ARM_LINK_회전-9
- removed joint LOWER_ARM_LINK미러_회전-11
- removed joint LOWER_ARM_LINK미러_회전-13
- removed joint TOP_ARM_LINK_회전-15
- removed joint TOP_ARM_LINK_회전-17
- removed joint TOP_ARM_LINK_회전-7
- removed joint TOP_ARM_LINK미러_회전-10
- removed joint TOP_ARM_LINK미러_회전-14
- removed joint TOP_ARM_LINK미러_회전-16
- removed joint wheel_leg_link_회전-1
- removed joint wheel_leg_link_회전-2
- removed joint wheel_leg_link_회전-3
- removed joint wheel_leg_link_회전-4
- removed joint wheel_leg_link_회전-5
- removed joint wheel_leg_link_회전-6
- added joint BODY_LINK_rev-18: type revolute, parent BODY_LINK, child LARGE_BEVEL_GEAR_LINK, origin xyz=0.25122109 0.0941 0.11559530000000001 rpy=3.141592653589793 1.42882689753879 3.141592653589793, axis 3.310086940655488e-08 0.0 0.9999997463849672, limit lower=-0.523599 upper=0.523599 effort=1000000 velocity=1000000
- added joint LOWER_ARM_LINK_MIR_rev-11: type continuous, parent LOWER_ARM_LINK_MIR, child wheel_leg_link, origin xyz=0.07940738 0.01623169 0.013999999999999999 rpy=-1.5707963267948966 -0.0 3.1010518807301253, axis 0.08099305115897235 0.0 -0.9967143433541829
- added joint LOWER_ARM_LINK_MIR_rev-13: type continuous, parent LOWER_ARM_LINK_MIR, child wheel_leg_link, origin xyz=-0.08046116000000002 0.009746949999999997 0.013999999999999999 rpy=-1.5707963267948966 -0.0 3.1010518807301253, axis 0.08099305115897235 0.0 -0.9967143433541829
- added joint LOWER_ARM_LINK_rev-8: type continuous, parent LOWER_ARM_LINK, child wheel_leg_link, origin xyz=0.07940738000000001 -0.016231690000000007 0.014000000000000021 rpy=1.5707963267948966 -0.0 3.1010518807301253, axis -3.447097470174465e-07 0.0 0.999999678291889
- added joint LOWER_ARM_LINK_rev-9: type continuous, parent LOWER_ARM_LINK, child wheel_leg_link, origin xyz=-0.08046116 -0.009746950000000006 0.014000000000000021 rpy=1.5707963267948966 -0.0 3.1010518807301253, axis -3.447097470174465e-07 0.0 0.999999678291889
- added joint TOP_ARM_LINK_MIR_rev-10: type continuous, parent TOP_ARM_LINK_MIR, child wheel_leg_link, origin xyz=0.09429581 -0.03938530999999999 0.16457262 rpy=1.5707963267948966 -0.0 0.0, axis 0.0 0.0 -0.9999999999999999
- added joint TOP_ARM_LINK_MIR_rev-14: type continuous, parent TOP_ARM_LINK_MIR, child LOWER_ARM_LINK_MIR, origin xyz=-0.14801959 -0.04386569 0.15057262 rpy=0.0 -0.0 0.0, axis 0.0 0.0 -1.0
- added joint TOP_ARM_LINK_MIR_rev-16: type continuous, parent TOP_ARM_LINK_MIR, child TOP_ARM_LINK, origin xyz=0.0 0.0 0.08514479 rpy=3.141592653589793 -0.0 0.0, axis 0.0 0.0 -1.0
- added joint TOP_ARM_LINK_rev-15: type continuous, parent TOP_ARM_LINK, child LOWER_ARM_LINK, origin xyz=-0.14801959 0.04386569 0.15057262 rpy=0.0 -0.0 0.0, axis 0.0 0.0 1.0
- added joint TOP_ARM_LINK_rev-17: type continuous, parent TOP_ARM_LINK, child TOP_ARM_LINK_MIR, origin xyz=0.0 0.0 0.08514479 rpy=3.141592653589793 -0.0 0.0, axis 0.0 0.0 1.0
- added joint TOP_ARM_LINK_rev-7: type continuous, parent TOP_ARM_LINK, child wheel_leg_link, origin xyz=0.09429581 0.03938530999999999 0.16457262 rpy=-1.5707963267948966 -0.0 0.0, axis 0.0 0.0 1.0
- added joint wheel_leg_link_rev-1: type continuous, parent wheel_leg_link, child wheel_link, origin xyz=-0.00015771000000000868 -0.005247629999999996 0.0808032 rpy=-1.5707963267948966 -0.0 3.1115479793871788, axis -1.634341986883614e-07 0.0 1.000000302500441
- added joint wheel_leg_link_rev-2: type continuous, parent wheel_leg_link, child wheel_link, origin xyz=-0.1661501764032297 0.01249438 0.08589107206261985 rpy=-1.5695778086865493 -0.0405224664905253 -0.0300693662642092, axis -2.5152151516851656e-05 -0.001218 0.999999551496584
- added joint wheel_leg_link_rev-3: type continuous, parent wheel_leg_link, child wheel_link, origin xyz=-0.32562453372237926 0.012494359999999998 0.07293224139610428 rpy=-1.5695778086865493 -0.0405224664905253 -0.0300693662642092, axis -2.5152151516851656e-05 -0.001218 0.999999551496584
- added joint wheel_leg_link_rev-4: type continuous, parent wheel_leg_link, child wheel_link, origin xyz=-0.0003754999999999953 0.23150607 0.0808032 rpy=-1.5707963267948966 -0.0 3.1115479793871788, axis -1.634341986883614e-07 0.0 1.000000302500441
- added joint wheel_leg_link_rev-5: type continuous, parent wheel_leg_link, child wheel_link, origin xyz=-0.1586477691654984 -0.23150607 0.09906585041123527 rpy=-1.572014844903244 0.04052246649052531 -0.030069366264209203, axis -2.5152151516851656e-05 -0.001218 0.999999551496584
- added joint wheel_leg_link_rev-6: type continuous, parent wheel_leg_link, child wheel_link, origin xyz=-0.31864777521112064 -0.23150607 0.09906585764015598 rpy=-1.572014844903244 0.04052246649052531 -0.030069366264209203, axis -2.5152151516851656e-05 -0.001218 0.999999551496584
